File: MCM-81349-MCM.kicad_sch (KiCad schematic)
At the start: 39 parts, among them J5 USB4105-GF-A, U5 ESP32-S3-WROOM-1-N16R8

Commit message: remove tbd
Parts:
- R22, R24: value TBD -> 9k53
- R23, R25: value TBD -> 430R
Changed lines of the file:
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@@
 			)
 		)
-		(property "Value" "TBD"
+		(property "Value" "430R"
 			(at 139.7 171.4499 0)
 			(effects
@@
 			)
 		)
-		(property "Description" "Resistor"
+		(property "Description" "RES 430 OHM 1% 1/16W 0402"
 			(at 137.16 170.18 0)
 			(effects
@@
 			)
 		)
-		(property "Value" "TBD"
+		(property "Value" "430R"
 			(at 101.6 171.4499 0)
 			(effects
@@
 			)
 		)
-		(property "Description" "Resistor"
+		(property "Description" "RES 430 OHM 1% 1/16W 0402"
 			(at 99.06 170.18 0)
 			(effects
@@
 			)
 		)
-		(property "Value" "TBD"
+		(property "Value" "9k53"
 			(at 139.7 161.2899 0)
 			(effects
@@
 			)
 		)
-		(property "Description" "Resistor"
+		(property "Description" "RES 9k53 OHM 1% 1/16W 0402"
 			(at 137.16 160.02 0)
 			(effects
@@
 			)
 		)
-		(property "Value" "TBD"
+		(property "Value" "9k53"
 			(at 101.6 161.2899 0)
 			(effects
@@
 			)
 		)
-		(property "Description" "Resistor"
+		(property "Description" "RES 9k53 OHM 1% 1/16W 0402"
 			(at 99.06 160.02 0)
 			(effects
